Commit message: feat: Add Gazebo simulation support for the robot, including new launch files, xacro definitions, and updated dependencies.

File: src/sme-4wcl-description/urdf/robot.urdf (robot description, URDF)
Before this commit: robot sme-4wcl, 9 links, 8 joints
Links:
- added link base_footprint
- link base_link: geometry collision mesh filename=package://sme-4wcl-description/meshes/base_plate_v2.stl; collision mesh filename=package://sme-4wcl-description/meshes/dcmotor_12v_v2.stl
- link base_top: geometry collision mesh filename=package://sme-4wcl-description/meshes/base_plate_top_v2.stl; visual mesh filename=package://sme-4wcl-description/meshes/base_plate_top_v2.stl
- link camera_1: geometry collision mesh filename=package://sme-4wcl-description/meshes/astra.stl; collision mesh filename=package://sme-4wcl-description/meshes/astra_clip1.stl
- link jetson_nano: geometry collision mesh filename=package://sme-4wcl-description/meshes/jetson_nano_v1.stl; visual mesh filename=package://sme-4wcl-description/meshes/jetson_nano_v1.stl
- link lidar_1: geometry collision mesh filename=package://sme-4wcl-description/meshes/ld19_bottom.stl; collision mesh filename=package://sme-4wcl-description/meshes/ld19_middle.stl
- link wheel_1: geometry collision mesh filename=package://sme-4wcl-description/meshes/part1.stl; collision mesh filename=package://sme-4wcl-description/meshes/part1.stl
- link wheel_2: geometry collision mesh filename=package://sme-4wcl-description/meshes/part1.stl; collision mesh filename=package://sme-4wcl-description/meshes/part1.stl
- link wheel_3: geometry collision mesh filename=package://sme-4wcl-description/meshes/part1.stl; collision mesh filename=package://sme-4wcl-description/meshes/part1.stl
- link wheel_4: geometry collision mesh filename=package://sme-4wcl-description/meshes/part1.stl; collision mesh filename=package://sme-4wcl-description/meshes/part1.stl
Joints:
- added joint base_footprint_joint: type fixed, parent base_footprint, child base_link, origin xyz=0 0 0 rpy=0 0 0

Commit message: Refactor mesh and RViz configuration paths by renaming the assets directory to meshes and relocating RViz files.

File: src/sme-4wcl-description/urdf/robot.urdf (robot description, URDF)
Before this commit: robot sme-4wcl, 10 links, 9 joints
Links:
- link base_link: geometry collision mesh filename=package://sme-4wcl-description/meshes/base_plate_v2.stl; collision mesh filename=package://sme-4wcl-description/meshes/dcmotor_12v_v2.stl
- link base_top: geometry collision mesh filename=package://sme-4wcl-description/meshes/base_plate_top_v2.stl; visual mesh filename=package://sme-4wcl-description/meshes/base_plate_top_v2.stl
- link camera_1: geometry collision mesh filename=package://sme-4wcl-description/meshes/astra.stl; collision mesh filename=package://sme-4wcl-description/meshes/astra_clip1.stl
- link jetson_nano: geometry collision mesh filename=package://sme-4wcl-description/meshes/jetson_nano_v1.stl; visual mesh filename=package://sme-4wcl-description/meshes/jetson_nano_v1.stl
- link lidar_1: geometry collision mesh filename=package://sme-4wcl-description/meshes/ld19_bottom.stl; collision mesh filename=package://sme-4wcl-description/meshes/ld19_middle.stl
- link wheel_1: geometry collision mesh filename=package://sme-4wcl-description/meshes/part1.stl; collision mesh filename=package://sme-4wcl-description/meshes/part1.stl
- link wheel_2: geometry collision mesh filename=package://sme-4wcl-description/meshes/part1.stl; collision mesh filename=package://sme-4wcl-description/meshes/part1.stl
- link wheel_3: geometry collision mesh filename=package://sme-4wcl-description/meshes/part1.stl; collision mesh filename=package://sme-4wcl-description/meshes/part1.stl
- link wheel_4: geometry collision mesh filename=package://sme-4wcl-description/meshes/part1.stl; collision mesh filename=package://sme-4wcl-description/meshes/part1.stl
