Commit message: refactor: rename package directories and update references to use underscores instead of hyphens.

File: src/sme_4wcl_description/urdf/robot.urdf (robot description, URDF)
Before this commit: robot sme-4wcl, 10 links, 9 joints
Links:
- link base_link: geometry collision mesh filename=package://sme_4wcl_description/meshes/base_plate_v2.stl; collision mesh filename=package://sme_4wcl_description/meshes/dcmotor_12v_v2.stl
- link base_top: geometry collision mesh filename=package://sme_4wcl_description/meshes/base_plate_top_v2.stl; visual mesh filename=package://sme_4wcl_description/meshes/base_plate_top_v2.stl
- link camera_1: geometry collision mesh filename=package://sme_4wcl_description/meshes/astra.stl; collision mesh filename=package://sme_4wcl_description/meshes/astra_clip1.stl
- link jetson_nano: geometry collision mesh filename=package://sme_4wcl_description/meshes/jetson_nano_v1.stl; visual mesh filename=package://sme_4wcl_description/meshes/jetson_nano_v1.stl
- link lidar_1: geometry collision mesh filename=package://sme_4wcl_description/meshes/ld19_bottom.stl; collision mesh filename=package://sme_4wcl_description/meshes/ld19_middle.stl
- link wheel_1: geometry collision mesh filename=package://sme_4wcl_description/meshes/part1.stl; collision mesh filename=package://sme_4wcl_description/meshes/part1.stl
- link wheel_2: geometry collision mesh filename=package://sme_4wcl_description/meshes/part1.stl; collision mesh filename=package://sme_4wcl_description/meshes/part1.stl
- link wheel_3: geometry collision mesh filename=package://sme_4wcl_description/meshes/part1.stl; collision mesh filename=package://sme_4wcl_description/meshes/part1.stl
- link wheel_4: geometry collision mesh filename=package://sme_4wcl_description/meshes/part1.stl; collision mesh filename=package://sme_4wcl_description/meshes/part1.stl

File: src/sme_4wcl_description/urdf/sme-4wcl.gazebo.xacro (robot description, xacro)
@@ -2,5 +2,5 @@
 <robot xmlns:xacro="http://www.ros.org/wiki/xacro" name="sme-4wcl">
   <!-- Include the generated URDF -->
-  <xacro:include filename="$(find sme-4wcl-description)/urdf/robot.urdf" />
+  <xacro:include filename="$(find sme_4wcl_description)/urdf/robot.urdf" />
   <!-- Gazebo physics properties for the wheels -->
   <gazebo reference="wheel_1">

File: src/sme_4wcl_description/urdf/sme-4wcl_classic.gazebo.xacro (robot description, xacro)
@@ -2,5 +2,5 @@
 <robot xmlns:xacro="http://www.ros.org/wiki/xacro" name="sme-4wcl">
   <!-- Include the generated URDF -->
-  <xacro:include filename="$(find sme-4wcl-description)/urdf/robot.urdf" />
+  <xacro:include filename="$(find sme_4wcl_description)/urdf/robot.urdf" />
   <!-- Gazebo physics properties for the wheels -->
   <gazebo reference="wheel_1">
