Commit message: refactor: Standardize URDF link naming, update Gazebo XACRO references, add IMU plugin, and include a new test world.

File: src/sme_4wcl_description/on-shape-export-urdf/sme_4wcl/robot.urdf (robot description, URDF)
Before this commit: robot sme-4wcl, 10 links, 9 joints
Links:
- removed link base_top
- removed link camera_1
- removed link jetson_nano
- removed link lidar_1
- removed link wheel_1
- removed link wheel_2
- removed link wheel_3
- removed link wheel_4
- added link base_top_link, mass 0.803036; collision mesh filename=package://assets/base_plate_top_v2.stl; visual mesh filename=package://assets/base_plate_top_v2.stl
- added link camera_1_link, mass 0.237529; collision mesh filename=package://assets/astra.stl; collision mesh filename=package://assets/astra_clip1.stl
- added link jetson_nano_link, mass 0.557665; collision mesh filename=package://assets/jetson_nano_v1.stl; visual mesh filename=package://assets/jetson_nano_v1.stl
- added link lidar_1_link, mass 0.0138375; collision mesh filename=package://assets/ld19_bottom.stl; collision mesh filename=package://assets/ld19_middle.stl
- added link wheel_1_link, mass 0.614542; collision mesh filename=package://assets/part1.stl; collision mesh filename=package://assets/part1.stl
- added link wheel_2_link, mass 0.614542; collision mesh filename=package://assets/part1.stl; collision mesh filename=package://assets/part1.stl
- added link wheel_3_link, mass 0.614542; collision mesh filename=package://assets/part1.stl; collision mesh filename=package://assets/part1.stl
- added link wheel_4_link, mass 0.614542; collision mesh filename=package://assets/part1.stl; collision mesh filename=package://assets/part1.stl
Joints:
- joint base_link_to_base_top: child base_top -> base_top_link
- joint base_link_to_jetson_nano: child jetson_nano -> jetson_nano_link
- joint base_link_to_wheel_1: child wheel_1 -> wheel_1_link
- joint base_link_to_wheel_2: child wheel_2 -> wheel_2_link
- joint base_link_to_wheel_3: child wheel_3 -> wheel_3_link
- joint base_link_to_wheel_4: child wheel_4 -> wheel_4_link
- joint base_top_to_camera_1: child camera_1 -> camera_1_link; parent base_top -> base_top_link
- joint base_top_to_lidar_1: child lidar_1 -> lidar_1_link; parent base_top -> base_top_link

File: src/sme_4wcl_description/urdf/robot.urdf (robot description, URDF)
Before this commit: robot sme-4wcl, 10 links, 9 joints
Links:
- removed link base_top
- removed link camera_1
- removed link jetson_nano
- removed link lidar_1
- removed link wheel_1
- removed link wheel_2
- removed link wheel_3
- removed link wheel_4
- added link base_top_link, mass 0.803036; collision mesh filename=package://sme_4wcl_description/meshes/base_plate_top_v2.stl; visual mesh filename=package://sme_4wcl_description/meshes/base_plate_top_v2.stl
- added link camera_1_link, mass 0.237529; collision mesh filename=package://sme_4wcl_description/meshes/astra.stl; collision mesh filename=package://sme_4wcl_description/meshes/astra_clip1.stl
- added link jetson_nano_link, mass 0.557665; collision mesh filename=package://sme_4wcl_description/meshes/jetson_nano_v1.stl; visual mesh filename=package://sme_4wcl_description/meshes/jetson_nano_v1.stl
- added link lidar_1_link, mass 0.0138375; collision mesh filename=package://sme_4wcl_description/meshes/ld19_bottom.stl; collision mesh filename=package://sme_4wcl_description/meshes/ld19_middle.stl
- added link wheel_1_link, mass 0.614542; collision mesh filename=package://sme_4wcl_description/meshes/part1.stl; collision mesh filename=package://sme_4wcl_description/meshes/part1.stl
- added link wheel_2_link, mass 0.614542; collision mesh filename=package://sme_4wcl_description/meshes/part1.stl; collision mesh filename=package://sme_4wcl_description/meshes/part1.stl
- added link wheel_3_link, mass 0.614542; collision mesh filename=package://sme_4wcl_description/meshes/part1.stl; collision mesh filename=package://sme_4wcl_description/meshes/part1.stl
- added link wheel_4_link, mass 0.614542; collision mesh filename=package://sme_4wcl_description/meshes/part1.stl; collision mesh filename=package://sme_4wcl_description/meshes/part1.stl
Joints:
- joint base_link_to_base_top: child base_top -> base_top_link
- joint base_link_to_jetson_nano: child jetson_nano -> jetson_nano_link
- joint base_link_to_wheel_1: child wheel_1 -> wheel_1_link
- joint base_link_to_wheel_2: child wheel_2 -> wheel_2_link
- joint base_link_to_wheel_3: child wheel_3 -> wheel_3_link
- joint base_link_to_wheel_4: child wheel_4 -> wheel_4_link
- joint base_top_to_camera_1: child camera_1 -> camera_1_link; parent base_top -> base_top_link
- joint base_top_to_lidar_1: child lidar_1 -> lidar_1_link; parent base_top -> base_top_link

File: src/sme_4wcl_description/urdf/sme-4wcl.gazebo.xacro (robot description, xacro)
@@ -4,5 +4,5 @@
   <xacro:include filename="$(find sme_4wcl_description)/urdf/robot.urdf" />
   <!-- Gazebo physics properties for the wheels -->
-  <gazebo reference="wheel_1">
+  <gazebo reference="wheel_1_link">
     <mu1>1.0</mu1>
     <mu2>1.0</mu2>
@@ -13,5 +13,5 @@
     <fdir1>1 0 0</fdir1>
   </gazebo>
-  <gazebo reference="wheel_2">
+  <gazebo reference="wheel_2_link">
     <mu1>1.0</mu1>
     <mu2>1.0</mu2>
@@ -22,5 +22,5 @@
     <fdir1>1 0 0</fdir1>
   </gazebo>
-  <gazebo reference="wheel_3">
+  <gazebo reference="wheel_3_link">
     <mu1>1.0</mu1>
     <mu2>1.0</mu2>
@@ -31,5 +31,5 @@
     <fdir1>1 0 0</fdir1>
   </gazebo>
-  <gazebo reference="wheel_4">
+  <gazebo reference="wheel_4_link">
     <mu1>1.0</mu1>
     <mu2>1.0</mu2>
@@ -69,9 +69,9 @@
       <joint_name>base_link_to_wheel_4</joint_name>
     </plugin>
-    <!-- Sensors Plugin -->
-    <plugin
-      filename="libignition-gazebo-imu-system.so"
+    <!-- IMU Plugin -->
+    <plugin filename="libignition-gazebo-imu-system.so"
       name="ignition::gazebo::systems::Imu">
     </plugin>
+    <!-- Sensors Plugin - Lidar-->
     <plugin
       filename="libignition-gazebo-sensors-system.so"
@@ -80,28 +80,30 @@
     </plugin>
   </gazebo>
-  <gazebo reference="lidar_1">
+  <!-- Lidar -->
+  <gazebo reference="lidar_1_link">
     <sensor name='gpu_lidar' type='gpu_lidar'>
-        <pose relative_to='lidar_1'>0 0 0 0 0 0</pose>
+        <pose>0 0 0 0 0 0</pose>
         <topic>/scan</topic>
+        <gz_frame_id>lidar_1_link</gz_frame_id>
         <update_rate>10</update_rate>
         <ray>
             <scan>
                 <horizontal>
-                    <samples>640</samples>
-                    <resolution>1</resolution>
-                    <min_angle>-1.396263</min_angle>
-                    <max_angle>1.396263</max_angle>
+                  <samples>640</samples>
+                  <resolution>1</resolution>
+                  <min_angle>0</min_angle>
+                  <max_angle>6.28318</max_angle>
                 </horizontal>
                 <vertical>
-                    <samples>1</samples>
-                    <resolution>0.01</resolution>
-                    <min_angle>0</min_angle>
-                    <max_angle>0</max_angle>
+                  <samples>1</samples>
+                  <resolution>0.01</resolution>
+                  <min_angle>0</min_angle>
+                  <max_angle>0</max_angle>
                 </vertical>
             </scan>
             <range>
-                <min>0.08</min>
-                <max>10.0</max>
-                <resolution>0.01</resolution>
+              <min>0.08</min>
+              <max>10.0</max>
+              <resolution>0.01</resolution>
             </range>
         </ray>
@@ -110,8 +112,9 @@
     </sensor>
   </gazebo>
-  <gazebo reference="jetson_nano">
-    <sensor name="jetson_nano" type="imu">
-      <gz_frame_id>jetson_nano</gz_frame_id>
-      <frame_id>jetson_nano</frame_id>
+  <!-- IMU -->
+  <gazebo reference="jetson_nano_link">
+    <sensor name="jetson_nano_imu" type="imu">
+      <gz_frame_id>jetson_nano_link</gz_frame_id>
+      <frame_id>jetson_nano_link</frame_id>
       <always_on>1</always_on>
       <update_rate>100</update_rate>

File: src/sme_4wcl_description/urdf/sme-4wcl_classic.gazebo.xacro (robot description, xacro)
@@ -4,5 +4,5 @@
   <xacro:include filename="$(find sme_4wcl_description)/urdf/robot.urdf" />
   <!-- Gazebo physics properties for the wheels -->
-  <gazebo reference="wheel_1">
+  <gazebo reference="wheel_1_link">
     <mu1>1.0</mu1>
     <mu2>1.0</mu2>
@@ -13,5 +13,5 @@
     <fdir1>1 0 0</fdir1>
   </gazebo>
-  <gazebo reference="wheel_2">
+  <gazebo reference="wheel_2_link">
     <mu1>1.0</mu1>
     <mu2>1.0</mu2>
@@ -22,5 +22,5 @@
     <fdir1>1 0 0</fdir1>
   </gazebo>
-  <gazebo reference="wheel_3">
+  <gazebo reference="wheel_3_link">
     <mu1>1.0</mu1>
     <mu2>1.0</mu2>
@@ -31,5 +31,5 @@
     <fdir1>1 0 0</fdir1>
   </gazebo>
-  <gazebo reference="wheel_4">
+  <gazebo reference="wheel_4_link">
     <mu1>1.0</mu1>
     <mu2>1.0</mu2>
@@ -80,5 +80,5 @@
     </plugin>
   </gazebo>
-  <gazebo reference="lidar_1">
+  <gazebo reference="lidar_1_link">
     <sensor name="lidar" type="ray">
       <always_on>true</always_on>
@@ -114,5 +114,5 @@
     </sensor>
   </gazebo>
-  <gazebo reference="jetson_nano">
+  <gazebo reference="jetson_nano_link">
     <sensor name="jetson_nano" type="imu">
       <always_on>true</always_on>

Commit message: feat: update robot description for sme_4wcl including URDF,, and mesh assets.

File: src/sme_4wcl_description/on-shape-export-urdf/sme_4wcl/robot.urdf (robot description, URDF)
Before this commit: robot sme_4wcl, 10 links, 9 joints
Links:
- link base_link: geometry collision mesh filename=package://assets\base_plate_v2.stl; collision mesh filename=package://assets\dcmotor_12v_v2.stl
- link base_top_link: geometry collision mesh filename=package://assets\base_plate_top_v2.stl; visual mesh filename=package://assets\base_plate_top_v2.stl
- link camera_1_link: geometry collision mesh filename=package://assets\astra.stl; collision mesh filename=package://assets\astra_clip1.stl
- link jetson_nano_link: geometry collision mesh filename=package://assets\jetson_nano_v1.stl; visual mesh filename=package://assets\jetson_nano_v1.stl
- link lidar_1_link: geometry collision mesh filename=package://assets\ld19_bottom.stl; collision mesh filename=package://assets\ld19_middle.stl
- link wheel_1_link: mass 0.614542 -> 0.228965; geometry collision mesh filename=package://assets\core.stl; collision mesh filename=package://assets\frame.stl
- link wheel_2_link: mass 0.614542 -> 0.228965; geometry collision mesh filename=package://assets\core__2.stl; collision mesh filename=package://assets\frame__2.stl
- link wheel_3_link: mass 0.614542 -> 0.228965; geometry collision mesh filename=package://assets\core__2.stl; collision mesh filename=package://assets\frame__2.stl
- link wheel_4_link: mass 0.614542 -> 0.228965; geometry collision mesh filename=package://assets\core.stl; collision mesh filename=package://assets\frame.stl
Joints:
- joint base_link_to_wheel_1: origin xyz=0.0750542 -0.106021 0.0175757 rpy=1.5708 -1.5708 0 -> xyz=0.0750542 -0.101021 0.0175757 rpy=1.5708 -1.5708 0
- joint base_link_to_wheel_2: origin xyz=0.074946 0.106022 0.0175757 rpy=1.5708 0 0 -> xyz=0.074946 0.101022 0.0175757 rpy=1.5708 -1.5708 0
- joint base_link_to_wheel_3: origin xyz=-0.0899458 -0.106021 0.0175757 rpy=1.5708 -1.5708 0 -> xyz=-0.0899458 -0.101021 0.0175757 rpy=1.5708 1.5708 0
- joint base_link_to_wheel_4: origin xyz=-0.090054 0.106022 0.0175757 rpy=1.5708 0 0 -> xyz=-0.090054 0.101022 0.0175757 rpy=1.5708 -1.5708 0

File: src/sme_4wcl_description/urdf/robot.urdf (robot description, URDF)
Before this commit: robot sme_4wcl, 10 links, 9 joints
Links:
- link base_link: geometry collision mesh filename=package://assets\base_plate_v2.stl; collision mesh filename=package://assets\dcmotor_12v_v2.stl
- link base_top_link: geometry collision mesh filename=package://assets\base_plate_top_v2.stl; visual mesh filename=package://assets\base_plate_top_v2.stl
- link camera_1_link: geometry collision mesh filename=package://assets\astra.stl; collision mesh filename=package://assets\astra_clip1.stl
- link jetson_nano_link: geometry collision mesh filename=package://assets\jetson_nano_v1.stl; visual mesh filename=package://assets\jetson_nano_v1.stl
- link lidar_1_link: geometry collision mesh filename=package://assets\ld19_bottom.stl; collision mesh filename=package://assets\ld19_middle.stl
- link wheel_1_link: mass 0.614542 -> 0.228965; geometry collision mesh filename=package://assets\core.stl; collision mesh filename=package://assets\frame.stl
- link wheel_2_link: mass 0.614542 -> 0.228965; geometry collision mesh filename=package://assets\core__2.stl; collision mesh filename=package://assets\frame__2.stl
- link wheel_3_link: mass 0.614542 -> 0.228965; geometry collision mesh filename=package://assets\core__2.stl; collision mesh filename=package://assets\frame__2.stl
- link wheel_4_link: mass 0.614542 -> 0.228965; geometry collision mesh filename=package://assets\core.stl; collision mesh filename=package://assets\frame.stl
Joints:
- joint base_link_to_wheel_1: origin xyz=0.0750542 -0.106021 0.0175757 rpy=1.5708 -1.5708 0 -> xyz=0.0750542 -0.101021 0.0175757 rpy=1.5708 -1.5708 0
- joint base_link_to_wheel_2: origin xyz=0.074946 0.106022 0.0175757 rpy=1.5708 0 0 -> xyz=0.074946 0.101022 0.0175757 rpy=1.5708 -1.5708 0
- joint base_link_to_wheel_3: origin xyz=-0.0899458 -0.106021 0.0175757 rpy=1.5708 -1.5708 0 -> xyz=-0.0899458 -0.101021 0.0175757 rpy=1.5708 1.5708 0
- joint base_link_to_wheel_4: origin xyz=-0.090054 0.106022 0.0175757 rpy=1.5708 0 0 -> xyz=-0.090054 0.101022 0.0175757 rpy=1.5708 -1.5708 0

Commit message: fix: urdf file for linux

File: src/sme_4wcl_description/on-shape-export-urdf/sme_4wcl/robot.urdf (robot description, URDF)
Before this commit: robot C:\GIT\sme\ROS\sme-4wcl\src\sme_4wcl_description\on-shape-export-urdf\sme_4wcl, 10 links, 9 joints
Links:
- link base_link: geometry collision mesh filename=package://assets/base_plate_v2.stl; collision mesh filename=package://assets/dcmotor_12v_v2.stl
- link base_top_link: geometry collision mesh filename=package://assets/base_plate_top_v2.stl; visual mesh filename=package://assets/base_plate_top_v2.stl
- link camera_1_link: geometry collision mesh filename=package://assets/astra.stl; collision mesh filename=package://assets/astra_clip1.stl
- link jetson_nano_link: geometry collision mesh filename=package://assets/jetson_nano_v1.stl; visual mesh filename=package://assets/jetson_nano_v1.stl
- link lidar_1_link: geometry collision mesh filename=package://assets/ld19_bottom.stl; collision mesh filename=package://assets/ld19_middle.stl
- link wheel_1_link: geometry collision mesh filename=package://assets/core.stl; collision mesh filename=package://assets/frame.stl
- link wheel_2_link: geometry collision mesh filename=package://assets/core__2.stl; collision mesh filename=package://assets/frame__2.stl
- link wheel_3_link: geometry collision mesh filename=package://assets/core__2.stl; collision mesh filename=package://assets/frame__2.stl
- link wheel_4_link: geometry collision mesh filename=package://assets/core.stl; collision mesh filename=package://assets/frame.stl

File: src/sme_4wcl_description/urdf/robot.urdf (robot description, URDF)
Before this commit: robot C:\GIT\sme\ROS\sme-4wcl\src\sme_4wcl_description\on-shape-export-urdf\sme_4wcl, 10 links, 9 joints
Links:
- link base_link: geometry collision mesh filename=package://sme_4wcl_description/meshes/base_plate_v2.stl; collision mesh filename=package://sme_4wcl_description/meshes/dcmotor_12v_v2.stl
- link base_top_link: geometry collision mesh filename=package://sme_4wcl_description/meshes/base_plate_top_v2.stl; visual mesh filename=package://sme_4wcl_description/meshes/base_plate_top_v2.stl
- link camera_1_link: geometry collision mesh filename=package://sme_4wcl_description/meshes/astra.stl; collision mesh filename=package://sme_4wcl_description/meshes/astra_clip1.stl
- link jetson_nano_link: geometry collision mesh filename=package://sme_4wcl_description/meshes/jetson_nano_v1.stl; visual mesh filename=package://sme_4wcl_description/meshes/jetson_nano_v1.stl
- link lidar_1_link: geometry collision mesh filename=package://sme_4wcl_description/meshes/ld19_bottom.stl; collision mesh filename=package://sme_4wcl_description/meshes/ld19_middle.stl
- link wheel_1_link: geometry collision mesh filename=package://sme_4wcl_description/meshes/core.stl; collision mesh filename=package://sme_4wcl_description/meshes/frame.stl
- link wheel_2_link: geometry collision mesh filename=package://sme_4wcl_description/meshes/core__2.stl; collision mesh filename=package://sme_4wcl_description/meshes/frame__2.stl
- link wheel_3_link: geometry collision mesh filename=package://sme_4wcl_description/meshes/core__2.stl; collision mesh filename=package://sme_4wcl_description/meshes/frame__2.stl
- link wheel_4_link: geometry collision mesh filename=package://sme_4wcl_description/meshes/core.stl; collision mesh filename=package://sme_4wcl_description/meshes/frame.stl
